Commit message: Update vitirover_gazebo.urdf
Added transform from robot to map.
Added joint_state_publisher plugin for rviz.

File: src/mobile_robot/urdf/vitirover_gazebo.urdf (robot description, URDF)
Before this commit: robot vitirover, 8 links, 7 joints
Links:
- added link map
- link base_footprint: geometry visual box size=0.001 0.001 0.001
Joints:
- added joint fixed: type fixed, parent map, child base_footprint, origin xyz=0 0 0 rpy=0 0 0

Commit message: Update vitirover_gazebo.urdf

File: src/mobile_robot/urdf/vitirover_gazebo.urdf (robot description, URDF)
Before this commit: robot vitirover, 9 links, 8 joints
Links:
- removed link map
- link base_footprint: geometry 
Joints:
- removed joint fixed
- joint front_left_wheel_joint: origin xyz=0.2 -0.1875 0.0 rpy=0 0 0 -> xyz=0.2 0.1875 0.0 rpy=0 0 0
- joint front_right_wheel_joint: origin xyz=0.2 0.1875 0.0 rpy=0 0 0 -> xyz=0.2 -0.1875 0.0 rpy=0 0 0
- joint rear_left_wheel_axle_joint: origin xyz=0 0 -0.1875 rpy=1.570796 0 0 -> xyz=0 0 0.1875 rpy=1.570796 0 0
- joint rear_right_wheel_axle_joint: origin xyz=0 0 0.1875 rpy=1.570796 0 0 -> xyz=0 0 -0.1875 rpy=1.570796 0 0
